File: pcb/pico-mediakeeb/pico-mediakeeb.kicad_pcb (KiCad board)
At the start: 2 copper layers, 10 parts, among them SW1 btn_prev, SW2 btn_play_pause, SW3 btn_next, SW4 btn_macro_1, SW5 btn_macro_2, SW6 btn_macro_3, SW7 Rotary_Encoder_Switch, U1 Pico

Commit message: Implement pcb design v1
Parts:
- removed SW7: Rotary_Encoder_Switch, Rotary_Encoder:RotaryEncoder_Alps_EC11E-Switch_Vertical_H20mm
- removed U1: Pico, Raspberry:RPi_Pico_SMD_TH
- added Pi Pico: , Raspberry:RPi_Pico_SMD_TH, F.Cu at (57.4, 78.0)
- added ROT_SW: Rotary_Encoder_Switch, Rotary_Encoder:RotaryEncoder_Alps_EC11E-Switch_Vertical_H20mm, F.Cu at (74.4, 74.6)
- moved R1 48.0 mm to (86.9, 80.5)
- moved SW6 36.4 mm to (99.8, 120.9)
- moved SW5 36.2 mm to (79.5, 120.9)
- moved SW3 36.0 mm to (99.8, 141.2)
- moved SW4 36.0 mm to (59.2, 120.9)
- moved SW2 35.8 mm to (79.5, 141.2)
- moved SW1 35.6 mm to (59.2, 141.2)
- moved R2 34.3 mm to (81.8, 87.6)
Routing:
- net Net-(R1-Pad1): track 212.3 -> 246.6 mm
- net Net-(SW7-PadC): track 6.51 -> 28.0 mm
- net Net-(R2-Pad2): track 64.6 -> 43.9 mm
- net Net-(SW3-Pad2): track 101.3 -> 84.9 mm
- net Net-(R1-Pad2): track 61.5 -> 46.2 mm
- net Net-(SW5-Pad2): track 33.6 -> 48.8 mm
- net Net-(SW6-Pad2): track 54.3 -> 68.9 mm
- net Net-(SW4-Pad2): track 15.2 -> 26.6 mm
- net Net-(SW2-Pad2): track 76.6 -> 65.7 mm
- net Net-(SW1-Pad2): track 48.9 -> 43.4 mm
- net Net-(SW7-PadS2): track 45.6 -> 41.4 mm
- net Net-(SW7-PadS1): track 40.5 -> 44.5 mm
Other:
- board outline added: 64.8 x 105.4 mm
- board text added: "10k"
- board text added: "GND"
- board text added: "PICO-MEDIAKEEB"
- board text added: "Version: 1.0 Author: Mircea Anton (Mike Anthony) https://github.com/mikeanth-dev/pico-mediakeeb"

Commit message: Update pcb traces and add JLC order number placeholder
Parts:
- SW1, SW2, SW3, SW4, SW5, SW6: footprint Button_Switch_Keyboard:SW_Cherry_MX_1.00u_Plate -> Button_Switch_Keyboard:SW_Cherry_MX_1.00u_PCB
Routing:
- net Net-(SW5-Pad2): track 48.8 -> 50.5 mm
- net Net-(SW2-Pad2): track 65.7 -> 67.0 mm
Other:
- board text added: "JLCJLCJLCJLC"
